File: EAGLE_files_2k17/eagle/DAq 2017_achyuth_new_teensy_v_2.0/DAq2017.brd (EAGLE design)
At the start: 191.1 x 124.5 mm, 51 parts, among them U2 PTN78000WAH

Commit message: Daq done; CAN ANalog has to be edited; RPM node also remains
Parts:
- moved SD_SS_PULLUP2 103.0 mm to (101.0, 7.94)
- moved SD_SS_PULLUP1 93.7 mm to (93.1, 6.76), turned to 270 degrees
- moved SD_SS_PULLUP 79.0 mm to (77.7, 13.4), turned to 90 degrees
- moved LCD 65.9 mm to (112.7, 29.8), turned to 0 degrees
- moved SD_CARD_FPC 56.1 mm to (116.2, 6.67), turned to 0 degrees
- moved TP4 44.8 mm to (58.1, 66.8)
- moved TP5 44.8 mm to (58.1, 59.9)
- moved SPLIT_C1 43.5 mm to (18.1, 12.1), turned to 180 degrees
- moved BULK_CER1 42.7 mm to (39.7, 12.1)
- moved BYPASS_CER1 42.7 mm to (37.1, 12.1)
- moved U$3 42.7 mm to (30.8, 12.1)
- moved SPLIT_R3 42.3 mm to (23.2, 10.8)
- moved SPLIT_R4 42.3 mm to (23.2, 13.3)
- moved 12V_OUT_LED 42.3 mm to (44.5, 79.1)
- moved R1 42.3 mm to (38.1, 79.1)
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Connections:
- removed net N$1: SD_SS_PULLUP2.1, U$1.22/A8
- net 12V: no longer U$1.VIN
- net 3V3: now also TESTPOINTS.1; no longer TESTPOINTS.8
- net 5V: now also LCD.P$3, TESTPOINTS.6, U$1.VIN; no longer LCD.P$1, TESTPOINTS.3
- net GND: now also TESTPOINTS.8; no longer TESTPOINTS.4
- net GPS_EN: now also SD_SS_PULLUP2.1, U$1.22/A8
- net LCD_RX: now also LCD.P$1; no longer LCD.P$3
- net MC_CAN_L: now also TESTPOINTS.3; no longer TESTPOINTS.1
- net SENSOR_CAN_H: now also TESTPOINTS.4; no longer TESTPOINTS.5
- net SENSOR_CAN_L: now also TESTPOINTS.5; no longer TESTPOINTS.6
Routing:
- net GND: track 33.0 -> 448.1 mm, vias 0 -> 13
- net 3V3: track 0.00 -> 253.4 mm, vias 0 -> 5
- net RESET: track 0.00 -> 181.4 mm, vias 0 -> 1
- net 5V: track 34.1 -> 206.5 mm, vias 0 -> 1
- net GPS_EN: track 0.00 -> 103.1 mm, vias 0 -> 3
- net GPS_FIX: track 0.00 -> 100.6 mm, vias 0 -> 1
- net RESET_CAN_NODE: track 0.00 -> 91.7 mm
- net LCD_RX: track 0.00 -> 70.9 mm
- net SENSOR_RX: track 0.00 -> 66.6 mm
- net SENSOR_TX: track 0.00 -> 65.2 mm
- net LCD_TX: track 0.00 -> 63.6 mm
- net 12V: track 0.00 -> 55.7 mm
- net RTC: track 0.00 -> 53.7 mm
- net 3.3V: track 0.00 -> 51.3 mm
- net SD_MISO: track 0.00 -> 49.4 mm
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- added copper zone on layer 16, net 3V3
- added copper zone on layer 16, net GND
Other:
- board size 191.1 x 124.5 mm -> 121.9 x 88.9 mm
