File: EAGLE_files_2k17/eagle/DAq 2017_achyuth_new_teensy_v_2.0/DAq2017.sch (EAGLE design)
At the start: 51 parts, among them U2 PTN78000WAH

Commit message: Daq done; CAN ANalog has to be edited; RPM node also remains
Connections:
- removed net N$1: SD_SS_PULLUP2.1, U$1.22/A8/T/PWM
- net 12V: no longer U$1.VIN
- net 3V3: now also TESTPOINTS.1; no longer TESTPOINTS.8
- net 5V: now also LCD.3, TESTPOINTS.6, U$1.VIN; no longer LCD.1, TESTPOINTS.3
- net GND: now also TESTPOINTS.8; no longer TESTPOINTS.4
- net GPS_EN: now also SD_SS_PULLUP2.1, U$1.22/A8/T/PWM
- net LCD_RX: now also LCD.1; no longer LCD.3
- net MC_CAN_L: now also TESTPOINTS.3; no longer TESTPOINTS.1
- net SENSOR_CAN_H: now also TESTPOINTS.4; no longer TESTPOINTS.5
- net SENSOR_CAN_L: now also TESTPOINTS.5; no longer TESTPOINTS.6
Other:
- moved on the sheet: TESTPOINTS, TP2, TP3, TP4, TP5
