File: EAGLE_files_2k17/eagle/CAN_node_analog/CAN_node_analog.brd (EAGLE design)
At the start: 160 x 100 mm, 15 parts

Commit message: Analog node done bitches :D, RPM will be done in 2 hrs :D #peace
Parts:
- SV1: device IIT_BOMBAY_Racing:FE05-1 -> con-lsta:FE06
- moved SV1 31.5 mm to (5.08, 32.7), turned to 270 degrees
- moved R2 11.1 mm to (39.1, 36.5)
- moved U$3 11.0 mm to (32.4, 42.2), turned to 90 degrees
- moved R4 9.92 mm to (39.1, 48.3), turned to 270 degrees
- moved R1 7.94 mm to (39.1, 30.8), turned to 90 degrees
- moved R3 4.26 mm to (39.1, 42.5)
Connections:
- net GND: now also SV1.6
Routing:
- net ANALOG_3: track 60.8 -> 118.2 mm
- net 5V: track 76.3 -> 102.9 mm, vias 3 -> 2
- net ANALOG_4: track 78.6 -> 102.9 mm, vias 1 -> 2
- net ANALOG_2: track 57.7 -> 73.9 mm
- net RESET_CAN_NODE: track 61.3 -> 46.9 mm, vias 1 -> 0
- net GND: track 91.4 -> 78.5 mm, vias 8 -> 6
- net ANALOG_IN_1: track 7.82 -> 16.3 mm
- net ANALOG_IN_2: track 15.9 -> 19.4 mm
- net ANALOG_1: track 64.0 -> 67.4 mm, vias 0 -> 1
- net ANALOG_IN_4: track 7.84 -> 5.43 mm
- net ANALOG_IN_3: track 15.3 -> 17.4 mm
- net CAN_L: track 32.7 -> 32.0 mm, vias 1 -> 0
- net 3V3: track 47.0 -> 46.6 mm, vias 2 -> 3

Commit message: All boards except SD Card is donegit add . will buy SD Card :D #peace
Parts:
- added LED1: (no value), IIT_BOMBAY_Racing:LED-1206
- added R10, R11, R12, R13, R14, R6, R7, R8, R9: (no value), IIT_BOMBAY_Racing:R0805
- moved R4 25.6 mm to (32.7, 23.5), turned to 180 degrees
- moved R3 3.86 mm to (38.4, 46.4)
- moved R1 1.42 mm to (38.4, 32.1)
- moved R2 0.90 mm to (38.4, 37.1)
Connections:
- new net N$1: LED1.C, R6.2
- new net N$2: R1.1, R7.1, R8.2, U$3.3
- new net N$3: R10.2, R2.1, R9.1, U$3.5
- new net N$4: R11.2, R3.1, R4.1, U$3.10
- new net N$6: R12.1, R13.1, R14.2, U$3.12
- net 3V3: now also R1.2, R12.2, R2.2, R3.2
- net 5V: no longer R1.2, R2.2, R3.2, R4.2
- net ANALOG_1: now also R7.2; no longer R1.1, U$3.3
- net ANALOG_2: now also R9.2; no longer R2.1, U$3.5
- net ANALOG_3: now also R4.2; no longer R3.1, U$3.10
- net ANALOG_4: now also R13.2; no longer R4.1, U$3.12
- net ANALOG_IN_3: now also U$3.13, U$3.14; no longer U$3.8, U$3.9
- net ANALOG_IN_4: now also U$3.8, U$3.9; no longer U$3.13, U$3.14
- net GND: now also R10.1, R11.1, R14.1, R6.1, R8.1
- net LED_OUT: now also LED1.A, U$1.11; no longer U$1.13
Routing:
- net ANALOG_3: track 118.2 -> 50.9 mm, vias 1 -> 0
- net ANALOG_4: track 102.9 -> 50.7 mm, vias 2 -> 0
- net GND: track 78.5 -> 130.2 mm, vias 6 -> 8
- net N$4: track 0.00 -> 43.6 mm, vias 0 -> 2
- net N$3: track 0.00 -> 41.3 mm
- net 3V3: track 46.6 -> 83.3 mm
- net N$6: track 0.00 -> 33.9 mm, vias 0 -> 2
- net N$2: track 0.00 -> 33.4 mm
- net ANALOG_1: track 67.4 -> 41.7 mm, vias 1 -> 0
- net ANALOG_2: track 73.9 -> 49.5 mm
- net LED_OUT: track 0.00 -> 15.6 mm
- net 5V: track 102.9 -> 90.0 mm, vias 2 -> 1
- net ANALOG_IN_4: track 5.43 -> 18.1 mm, vias 0 -> 1
- net ANALOG_IN_3: track 17.4 -> 6.22 mm
- net ANALOG_IN_1: track 16.3 -> 13.9 mm
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