File: EAGLE_files_2k17/eagle/CAN_node_analog/CAN_node_analog.sch (EAGLE design)
At the start: 14 parts

Commit message: Daq done; CAN ANalog has to be edited; RPM node also remains
Parts:
- added SV1: (no value), IIT_BOMBAY_Racing:FE05-1
Connections:
- removed net N$1: U$3A.-IN, U$3A.OUT
- removed net N$12: X1.9
- removed net N$13: X1.10
- removed net N$2: U$3B.-IN, U$3B.OUT
- removed net N$3: U$3C.-IN, U$3C.OUT
- removed net N$4: U$3D.-IN, U$3D.OUT
- new net RESET_CAN_NODE: SV1.1, X1.10
- net ANALOG_1: now also SV1.5, X1.6; no longer X1.5
- net ANALOG_2: now also SV1.4, X1.7; no longer X1.6
- net ANALOG_3: now also SV1.3, X1.8; no longer X1.7
- net ANALOG_4: now also SV1.2, X1.9; no longer X1.8
- net ANALOG_IN_1: now also U$3A.-IN, U$3A.OUT
- net ANALOG_IN_2: now also U$3B.-IN, U$3B.OUT
- net ANALOG_IN_3: now also U$3C.-IN, U$3C.OUT
- net ANALOG_IN_4: now also U$3D.-IN, U$3D.OUT
Changed lines of the file:
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@@
 <part name="R4" library="IIT_BOMBAY_Racing" deviceset="R-EU_" device="R0805"/>
 <part name="R1" library="IIT_BOMBAY_Racing" deviceset="R-EU_" device="R0805"/>
+<part name="SV1" library="IIT_BOMBAY_Racing" deviceset="FE05-1" device=""/>
 </parts>
 <sheets>
@@
 <instance part="R4" gate="G$1" x="-33.02" y="7.62" rot="R90"/>
 <instance part="R1" gate="G$1" x="-33.02" y="78.74" rot="R90"/>
+<instance part="SV1" gate="G$1" x="187.96" y="45.72"/>
 </instances>
 <busses>
@@
 <label x="76.2" y="55.88" size="1.778" layer="95"/>
 </segment>
+<segment>
+<pinref part="U$3" gate="A" pin="-IN"/>
+<wire x1="-22.86" y1="68.58" x2="-27.94" y2="68.58" width="0.1524" layer="91"/>
+<wire x1="-27.94" y1="68.58" x2="-27.94" y2="58.42" width="0.1524" layer="91"/>
+<wire x1="-27.94" y1="58.42" x2="0" y2="58.42" width="0.1524" layer="91"/>
+<wire x1="0" y1="58.42" x2="0" y2="71.12" width="0.1524" layer="91"/>
+<pinref part="U$3" gate="A" pin="OUT"/>
+<wire x1="0" y1="71.12" x2="-7.62" y2="71.12" width="0.1524" layer="91"/>
+<wire x1="0" y1="71.12" x2="10.16" y2="71.12" width="0.1524" layer="91"/>
+<label x="15.24" y="71.12" size="1.778" layer="95" xref="yes"/>
+</segment>
 </net>
 <net name="ANALOG_IN_2" class="0">
@@
 <label x="76.2" y="53.34" size="1.778" layer="95"/>
 </segment>
+<segment>
+<pinref part="U$3" gate="B" pin="-IN"/>
+<wire x1="-22.86" y1="45.72" x2="-27.94" y2="45.72" width="0.1524" layer="91"/>
+<wire x1="-27.94" y1="45.72" x2="-27.94" y2="35.56" width="0.1524" layer="91"/>
+<wire x1="-27.94" y1="35.56" x2="0" y2="35.56" width="0.1524" layer="91"/>
+<wire x1="0" y1="35.56" x2="0" y2="48.26" width="0.1524" layer="91"/>
+<pinref part="U$3" gate="B" pin="OUT"/>
+<wire x1="0" y1="48.26" x2="-7.62" y2="48.26" width="0.1524" layer="91"/>
+<wire x1="0" y1="48.26" x2="10.16" y2="48.26" width="0.1524" layer="91"/>
+<label x="15.24" y="48.26" size="1.778" layer="95" xref="yes"/>
+</segment>
 </net>
 <net name="ANALOG_IN_3" class="0">
@@
 <label x="76.2" y="50.8" size="1.778" layer="95"/>
 </segment>
+<segment>
+<pinref part="U$3" gate="C" pin="-IN"/>
+<wire x1="-22.86" y1="22.86" x2="-27.94" y2="22.86" width="0.1524" layer="91"/>
+<wire x1="-27.94" y1="22.86" x2="-27.94" y2="12.7" width="0.1524" layer="91"/>
+<wire x1="-27.94" y1="12.7" x2="0" y2="12.7" width="0.1524" layer="91"/>
+<wire x1="0" y1="12.7" x2="0" y2="25.4" width="0.1524" layer="91"/>
+<pinref part="U$3" gate="C" pin="OUT"/>
+<wire x1="0" y1="25.4" x2="-7.62" y2="25.4" width="0.1524" layer="91"/>
+<wire x1="0" y1="25.4" x2="10.16" y2="25.4" width="0.1524" layer="91"/>
+<label x="15.24" y="25.4" size="1.778" layer="95" xref="yes"/>
+</segment>
 </net>
 <net name="ANALOG_IN_4" class="0">
@@
 <wire x1="104.14" y1="48.26" x2="91.44" y2="48.26" width="0.1524" layer="91"/>
 <label x="76.2" y="48.26" size="1.778" layer="95"/>
+</segment>
+<segment>
+<pinref part="U$3" gate="D" pin="-IN"/>
+<wire x1="-22.86" y1="-2.54" x2="-27.94" y2="-2.54" width="0.1524" layer="91"/>
+<wire x1="-27.94" y1="-2.54" x2="-27.94" y2="-12.7" width="0.1524" layer="91"/>
+<wire x1="-27.94" y1="-12.7" x2="0" y2="-12.7" width="0.1524" layer="91"/>
+<wire x1="0" y1="-12.7" x2="0" y2="0" width="0.1524" layer="91"/>
+<pinref part="U$3" gate="D" pin="OUT"/>
+<wire x1="0" y1="0" x2="-7.62" y2="0" width="0.1524" layer="91"/>
+<wire x1="0" y1="0" x2="10.16" y2="0" width="0.1524" layer="91"/>
+<label x="15.24" y="0" size="1.778" layer="95" xref="yes"/>
 </segment>
 </net>
@@
 <net name="ANALOG_1" class="0">
 <segment>
-<pinref part="X1" gate="G$1" pin="5"/>
-<wire x1="231.14" y1="53.34" x2="223.52" y2="53.34" width="0.1524" layer="91"/>
-<label x="208.28" y="53.34" size="1.778" layer="95"/>
-</segment>
-<segment>
 <pinref part="U$3" gate="A" pin="+IN"/>
 <wire x1="-22.86" y1="73.66" x2="-33.02" y2="73.66" width="0.1524" layer="91"/>
@@
 <junction x="-33.02" y="73.66"/>
 </segment>
+<segment>
+<pinref part="X1" gate="G$1" pin="6"/>
+<wire x1="231.14" y1="50.8" x2="195.58" y2="50.8" width="0.1524" layer="91"/>
+<label x="208.28" y="50.8" size="1.778" layer="95"/>
+<pinref part="SV1" gate="G$1" pin="5"/>
+</segment>
 </net>
 <net name="ANALOG_2" class="0">
-<segment>
-<pinref part="X1" gate="G$1" pin="6"/>
-<wire x1="231.14" y1="50.8" x2="223.52" y2="50.8" width="0.1524" layer="91"/>
-<label x="208.28" y="50.8" size="1.778" layer="95"/>
-</segment>
 <segment>
 <pinref part="U$3" gate="B" pin="+IN"/>
@@
 <junction x="-33.02" y="50.8"/>
 </segment>
+<segment>
+<pinref part="X1" gate="G$1" pin="7"/>
+<wire x1="231.14" y1="48.26" x2="195.58" y2="48.26" width="0.1524" layer="91"/>
+<label x="208.28" y="48.26" size="1.778" layer="95"/>
+<pinref part="SV1" gate="G$1" pin="4"/>
+</segment>
 </net>
 <net name="ANALOG_3" class="0">
-<segment>
-<pinref part="X1" gate="G$1" pin="7"/>
-<wire x1="231.14" y1="48.26" x2="223.52" y2="48.26" width="0.1524" layer="91"/>
-<label x="208.28" y="48.26" size="1.778" layer="95"/>
-</segment>
 <segment>
 <pinref part="U$3" gate="C" pin="+IN"/>
@@
 <junction x="-33.02" y="27.94"/>
 </segment>
+<segment>
+<pinref part="X1" gate="G$1" pin="8"/>
+<wire x1="231.14" y1="45.72" x2="195.58" y2="45.72" width="0.1524" layer="91"/>
+<label x="208.28" y="45.72" size="1.778" layer="95"/>
+<pinref part="SV1" gate="G$1" pin="3"/>
+</segment>
 </net>
 <net name="ANALOG_4" class="0">
-<segment>
-<pinref part="X1" gate="G$1" pin="8"/>
-<wire x1="231.14" y1="45.72" x2="223.52" y2="45.72" width="0.1524" layer="91"/>
-<label x="208.28" y="45.72" size="1.778" layer="95"/>
-</segment>
 <segment>
 <pinref part="U$3" gate="D" pin="+IN"/>
@@
 <wire x1="-33.02" y1="2.54" x2="-22.86" y2="2.54" width="0.1524" layer="91"/>
 <junction x="-33.02" y="2.54"/>
+</segment>
+<segment>
+<pinref part="X1" gate="G$1" pin="9"/>
+<wire x1="231.14" y1="43.18" x2="195.58" y2="43.18" width="0.1524" layer="91"/>
+<label x="208.28" y="43.18" size="1.778" layer="95"/>
+<pinref part="SV1" gate="G$1" pin="2"/>
 </segment>
 </net>
@@
 </segment>
 </net>
-<net name="N$12" class="0">
-<segment>
-<pinref part="X1" gate="G$1" pin="9"/>
-<wire x1="231.14" y1="43.18" x2="223.52" y2="43.18" width="0.1524" layer="91"/>
-</segment>
-</net>
-<net name="N$13" class="0">
+<net name="RESET_CAN_NODE" class="0">
 <segment>
 <pinref part="X1" gate="G$1" pin="10"/>
-<wire x1="231.14" y1="40.64" x2="223.52" y2="40.64" width="0.1524" layer="91"/>
+<pinref part="SV1" gate="G$1" pin="1"/>
+<wire x1="231.14" y1="40.64" x2="195.58" y2="40.64" width="0.1524" layer="91"/>
+<label x="203.2" y="40.64" size="1.778" layer="95"/>
 </segment>
 </net>
@@
 </segment>
 </net>
-<net name="N$1" class="0">
-<segment>
-<pinref part="U$3" gate="A" pin="-IN"/>
-<wire x1="-22.86" y1="68.58" x2="-27.94" y2="68.58" width="0.1524" layer="91"/>
-<wire x1="-27.94" y1="68.58" x2="-27.94" y2="58.42" width="0.1524" layer="91"/>
-<wire x1="-27.94" y1="58.42" x2="0" y2="58.42" width="0.1524" layer="91"/>
-<wire x1="0" y1="58.42" x2="0" y2="71.12" width="0.1524" layer="91"/>
-<pinref part="U$3" gate="A" pin="OUT"/>
-<wire x1="0" y1="71.12" x2="-7.62" y2="71.12" width="0.1524" layer="91"/>
-<wire x1="0" y1="71.12" x2="10.16" y2="71.12" width="0.1524" layer="91"/>
-</segment>
-</net>
-<net name="N$2" class="0">
-<segment>
-<pinref part="U$3" gate="B" pin="-IN"/>
-<wire x1="-22.86" y1="45.72" x2="-27.94" y2="45.72" width="0.1524" layer="91"/>
-<wire x1="-27.94" y1="45.72" x2="-27.94" y2="35.56" width="0.1524" layer="91"/>
-<wire x1="-27.94" y1="35.56" x2="0" y2="35.56" width="0.1524" layer="91"/>
-<wire x1="0" y1="35.56" x2="0" y2="48.26" width="0.1524" layer="91"/>
-<pinref part="U$3" gate="B" pin="OUT"/>
-<wire x1="0" y1="48.26" x2="-7.62" y2="48.26" width="0.1524" layer="91"/>
-<wire x1="0" y1="48.26" x2="10.16" y2="48.26" width="0.1524" layer="91"/>
-</segment>
-</net>
-<net name="N$3" class="0">
-<segment>
-<pinref part="U$3" gate="C" pin="-IN"/>
-<wire x1="-22.86" y1="22.86" x2="-27.94" y2="22.86" width="0.1524" layer="91"/>
-<wire x1="-27.94" y1="22.86" x2="-27.94" y2="12.7" width="0.1524" layer="91"/>
-<wire x1="-27.94" y1="12.7" x2="0" y2="12.7" width="0.1524" layer="91"/>
-<wire x1="0" y1="12.7" x2="0" y2="25.4" width="0.1524" layer="91"/>
-<pinref part="U$3" gate="C" pin="OUT"/>
-<wire x1="0" y1="25.4" x2="-7.62" y2="25.4" width="0.1524" layer="91"/>
-<wire x1="0" y1="25.4" x2="10.16" y2="25.4" width="0.1524" layer="91"/>
-</segment>
-</net>
-<net name="N$4" class="0">
-<segment>
-<pinref part="U$3" gate="D" pin="-IN"/>
-<wire x1="-22.86" y1="-2.54" x2="-27.94" y2="-2.54" width="0.1524" layer="91"/>
-<wire x1="-27.94" y1="-2.54" x2="-27.94" y2="-12.7" width="0.1524" layer="91"/>
-<wire x1="-27.94" y1="-12.7" x2="0" y2="-12.7" width="0.1524" layer="91"/>
-<wire x1="0" y1="-12.7" x2="0" y2="0" width="0.1524" layer="91"/>
-<pinref part="U$3" gate="D" pin="OUT"/>
-<wire x1="0" y1="0" x2="-7.62" y2="0" width="0.1524" layer="91"/>
-<wire x1="0" y1="0" x2="10.16" y2="0" width="0.1524" layer="91"/>
-</segment>
-</net>

Commit message: Analog node done bitches :D, RPM will be done in 2 hrs :D #peace
Parts:
- SV1: device IIT_BOMBAY_Racing:FE05-1 -> con-lsta:FE06-1
Connections:
- net GND: now also SV1.6
Changed lines of the file:
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@@
 <part name="R4" library="IIT_BOMBAY_Racing" deviceset="R-EU_" device="R0805"/>
 <part name="R1" library="IIT_BOMBAY_Racing" deviceset="R-EU_" device="R0805"/>
-<part name="SV1" library="IIT_BOMBAY_Racing" deviceset="FE05-1" device=""/>
+<part name="SV1" library="con-lsta" deviceset="FE06-1" device=""/>
 </parts>
 <sheets>
@@
 <instance part="R4" gate="G$1" x="-33.02" y="7.62" rot="R90"/>
 <instance part="R1" gate="G$1" x="-33.02" y="78.74" rot="R90"/>
-<instance part="SV1" gate="G$1" x="187.96" y="45.72"/>
+<instance part="SV1" gate="G$1" x="190.5" y="45.72"/>
 </instances>
 <busses>
@@
 <pinref part="GND1" gate="1" pin="GND"/>
 </segment>
+<segment>
+<wire x1="198.12" y1="53.34" x2="208.28" y2="53.34" width="0.1524" layer="91"/>
+<label x="203.2" y="53.34" size="1.778" layer="95"/>
+<pinref part="SV1" gate="G$1" pin="6"/>
+</segment>
 </net>
 <net name="ANALOG_1" class="0">
@@
 <segment>
 <pinref part="X1" gate="G$1" pin="6"/>
-<wire x1="231.14" y1="50.8" x2="195.58" y2="50.8" width="0.1524" layer="91"/>
+<wire x1="231.14" y1="50.8" x2="198.12" y2="50.8" width="0.1524" layer="91"/>
 <label x="208.28" y="50.8" size="1.778" layer="95"/>
 <pinref part="SV1" gate="G$1" pin="5"/>
@@
 <segment>
 <pinref part="X1" gate="G$1" pin="7"/>
-<wire x1="231.14" y1="48.26" x2="195.58" y2="48.26" width="0.1524" layer="91"/>
+<wire x1="231.14" y1="48.26" x2="198.12" y2="48.26" width="0.1524" layer="91"/>
 <label x="208.28" y="48.26" size="1.778" layer="95"/>
 <pinref part="SV1" gate="G$1" pin="4"/>
@@
 <segment>
 <pinref part="X1" gate="G$1" pin="8"/>
-<wire x1="231.14" y1="45.72" x2="195.58" y2="45.72" width="0.1524" layer="91"/>
+<wire x1="231.14" y1="45.72" x2="198.12" y2="45.72" width="0.1524" layer="91"/>
 <label x="208.28" y="45.72" size="1.778" layer="95"/>
 <pinref part="SV1" gate="G$1" pin="3"/>
@@
 <segment>
 <pinref part="X1" gate="G$1" pin="9"/>
-<wire x1="231.14" y1="43.18" x2="195.58" y2="43.18" width="0.1524" layer="91"/>
+<wire x1="231.14" y1="43.18" x2="198.12" y2="43.18" width="0.1524" layer="91"/>
 <label x="208.28" y="43.18" size="1.778" layer="95"/>
 <pinref part="SV1" gate="G$1" pin="2"/>
@@
 <segment>
 <pinref part="X1" gate="G$1" pin="10"/>
+<wire x1="231.14" y1="40.64" x2="198.12" y2="40.64" width="0.1524" layer="91"/>
+<label x="203.2" y="40.64" size="1.778" layer="95"/>
 <pinref part="SV1" gate="G$1" pin="1"/>
-<wire x1="231.14" y1="40.64" x2="195.58" y2="40.64" width="0.1524" layer="91"/>
-<label x="203.2" y="40.64" size="1.778" layer="95"/>
-</segment>
-</net>
+</segment>
+</net>

Commit message: All boards except SD Card is donegit add . will buy SD Card :D #peace
Parts:
- added LED1: (no value), IIT_BOMBAY_Racing:LED1206
- added R10, R11, R12, R13, R14, R6, R7, R8, R9: (no value), IIT_BOMBAY_Racing:R-EU_R0805
Connections:
- new net N$1: LED1.C, R6.2
- new net N$2: R1.1, R7.1, R8.2, U$3A.+IN
- new net N$3: R10.2, R2.1, R9.1, U$3B.+IN
- new net N$4: R11.2, R3.1, R4.1, U$3C.+IN
- new net N$6: R12.1, R13.1, R14.2, U$3D.+IN
- net 3V3: now also R1.2, R12.2, R2.2, R3.2
- net 5V: no longer R1.2, R2.2, R3.2, R4.2
- net ANALOG_1: now also R7.2; no longer R1.1, U$3A.+IN
- net ANALOG_2: now also R9.2; no longer R2.1, U$3B.+IN
- net ANALOG_3: now also R4.2; no longer R3.1, U$3C.+IN
- net ANALOG_4: now also R13.2; no longer R4.1, U$3D.+IN
- net ANALOG_IN_3: now also U$3D.-IN, U$3D.OUT; no longer U$3C.-IN, U$3C.OUT
- net ANALOG_IN_4: now also U$3C.-IN, U$3C.OUT; no longer U$3D.-IN, U$3D.OUT
- net GND: now also R10.1, R11.1, R14.1, R6.1, R8.1
- net LED_OUT: now also LED1.A, U$1.11/MOSI; no longer U$1.13/SCK/LED
Other:
- moved on the sheet: R4
