File: EAGLE_files_2k17/eagle/CAN_node_rpm_f2v/CAN_node_rpm_f2v.sch (EAGLE design)
At the start: 29 parts, among them IC1 MICROCHIP_PIC18F2580-I/ML, IC2 LM1117IMPX-ADJ, Q1 CSM-7X-DU, U1 TEXAS-INSTRUMENTS_BY_ELEMENT1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

Commit message: All boards except SD Card is donegit add . will buy SD Card :D #peace
Parts:
- removed C1, C2, C4: 22pF, resistor:C-USC0805
- removed C3, C6: 10uF, resistor:C-EUC0805
- removed C5: (no value), rcl:CPOL-EUSMCA
- removed CONNECTOR_PINS: (no value), con-lstb:MA04-2
- removed F1: 6V/0.5A, sparkfun_fuses:PPTC_HALF-AMP
- removed IC1: MICROCHIP_PIC18F2580-I/ML, IITBRacing_CAN_node_Evo5:MICROCHIP_PIC18F2580-I/ML
- removed IC2: LM1117IMPX-ADJ, lm1117:LM1117IMPX-ADJ
- removed LED2: (no value), IITBRacing_CAN_node_Evo5:LED_LED5MM
- removed LM1: 7372, 7372:7372
- removed Q1: CSM-7X-DU, crystal:CSM-7X-DU
- removed R10, R11, R6: 4k7, resistor:R-EU_R0805
- removed R14, R3: 5M1, resistor:R-EU_R0805
- removed R15, R4: 3M6, resistor:R-EU_R0805
- removed R2: 47K, resistor:R-EU_R0805
- removed R7: 470, resistor:R-EU_R0805
- removed R8: 10k, resistor:R-EU_R0805
- removed R9: 1k, resistor:R-EU_R0805
- added BULK_CER: 10uF, LV:C-EUC0805
- added BYPASS_CER: 100nF, LV:C-EUC0805
- added SPLIT_C: 4n7F, LV:C-EUC0805
- added SPLIT_R1, SPLIT_R2: 60E, LV:R-EU_R0805
- added U$1: TEENSY_3.1_BASIC, IIT_BOMBAY_Racing:TEENSY_3.1_BASIC
- added U$2: SN65HVD230/1, texas_1:SN65HVD230/1
- added X1: (no value), IIT_BOMBAY_Racing:HEADER_POS8_43045-0812
- LED1: device IITBRacing_CAN_node_Evo5:LED_LED5MM -> IITBRacing_CAN_node_Evo5:LED_LEDSMT1206
- R1: value 47K -> (none)
- R5: value 1k -> 4K7; device resistor:R-EU_R0805 -> LV:R-EU_R0805
- SV1: device con-lstb:MA06-1 -> con-lsta:FE05-1
- U1: value TEXAS-INSTRUMENTS_BY_ELEMENT14_BATCH_1_SN65HVD1050D -> TL082ID; device IITBRacing_CAN_node_Evo5:TEXAS-INSTRUMENTS_BY_ELEMENT14_BATCH_1_SN65HVD1050D -> Texas Instruments_By_element14_Batch_1:TL082ID
Connections:
- removed net CAN_RX: IC1.CANRX/RB3, U1.RXD
- removed net CAN_TX: IC1.INT2/CANTX/RB2, U1.TXD
- removed net DIG_IN0: IC1.INT0/AN10/RB0, R14.2, R15.1
- removed net DIG_IN1: IC1.INT1/AN8/RB1, R3.2, R4.1
- removed net LED: IC1.RC2/CCP1, R5.2
- removed net MCLR: IC1.RE3/!MCLR/VPP, R7.1, SV1.1
- removed net N$10: LM1.-IN_B, LM1.OUT_B, R14.1
- removed net N$2: R6.2, U1.S
- removed net N$3: C4.1, R7.2, R8.1
- removed net N$4: F1.1, IC2.IN
- removed net N$7: C6.1, R10.2, R11.1
- removed net N$8: LM1.-IN_A, LM1.OUT_A, R3.1
- removed net OSC1: C2.1, IC1.RA7/CLKI/OSC1, Q1.1
- removed net OSC2: C1.1, IC1.RA6/CLKO/OSC2, Q1.2
- removed net PGC: IC1.KBI2/PGC/RB6, SV1.5
- removed net PGD: IC1.KBI3/PGD/RB7, SV1.4
- removed net PGM: IC1.KBI1/PGM/RB5, SV1.6
- removed net RPM_IN_0: CONNECTOR_PINS.2, LM1.+IN_B, R2.2
- removed net VCAP: C3.1, IC1.RA4/T0CKI
- new net 3V3: BULK_CER.1, BYPASS_CER.1, U$1.3.3V, U$2.VCC
- new net LED_OUT: R1.2, U$1.11/MOSI
- new net N$9: SPLIT_C.1, SPLIT_R1.2, SPLIT_R2.2, U$2.VREF
- new net RESET_CAN_NODE: SV1.1, X1.8
- new net RPM_1: SV1.3, U1.1IN+, X1.6
- new net RPM_2: SV1.2, U1.2IN+, X1.7
- new net RPM_IN_2: U$1.7/RX3, U1.2IN-, U1.2OUT
- new net UC_RX: U$1.4/CAN-RX-PWM, U$2.R
- new net UC_TX: U$1.3/CAN-TX/PWM, U$2.D
- net 12V: now also U1.VCC+, X1.5; no longer CONNECTOR_PINS.8, F1.2, LM1.V+, R1.1, R2.1, R9.2
- net 5V: now also U$1.VIN, X1.1; no longer C5.+, CONNECTOR_PINS.6, IC1.VDD, IC2.OUT, IC2.OUT1, R8.2, SV1.2, U1.VCC
- net CAN_H: now also SPLIT_R1.1, U$2.CANH, X1.3; no longer CONNECTOR_PINS.3, R11.2, U1.CANH
- net CAN_L: now also SPLIT_R2.1, U$2.CANL, X1.4; no longer CONNECTOR_PINS.1, R10.1, U1.CANL
- net GND: now also BULK_CER.2, BYPASS_CER.2, R5.1, SPLIT_C.2, SV1.4, SV1.5, U$1.AGND, U$1.GND, U$2.GND, U1.VCC-, X1.2; no longer C1.2, C2.2, C3.2, C4.2, C5.-, C6.2, CONNECTOR_PINS.5, CONNECTOR_PINS.7, IC1.VSS@1, IC2.ADJ, LED2.C, LM1.V-, R15.2, R4.2, R6.1, SV1.3, U1.GND
- net N$1: now also R1.1; no longer R5.1
- net N$5: now also R5.2, U$2.RS; no longer LED2.A, R9.1
- net RPM_IN_1: now also U$1.6/PWM, U1.1IN-, U1.1OUT; no longer CONNECTOR_PINS.4, LM1.+IN_A, R1.2
Other:
- note removed: "LM1117 5V"
- note removed: "OPAMP 7372"
- note removed: "PIC18F25K80"
- note removed: "PROGRAM PINS"
- note removed: "SN65HVD1050"
- moved on the sheet: LED1, R1, R5, U1
